Commit message: stiff robot

File: assets/franka/panda.urdf (robot description, URDF)
Before this commit: robot panda, 12 links, 11 joints
Links:
- link panda_hand: mass None -> 0.646926
- link panda_leftfinger: mass None -> 0.646926
- link panda_link0: mass None -> 0.646926
- link panda_link8: mass 0.0 -> 3.0
- link panda_rightfinger: mass None -> 0.646926
Joints:
- removed joint panda_finger_joint1
- removed joint panda_finger_joint2
